Commit message: gazebo

File: turtlebot_gazebo/urdf/turtlebot3_burger_artag.urdf.xacro (robot description, xacro)
@@ -164,3 +164,36 @@
       <child link="artag"/>
     </joint>
+    <link name='light_link'>
+        <visual name='light_source'>
+          <pose>0 0 0 0 0 0</pose>
+          <geometry>
+            <sphere>
+              <radius>0.025</radius>
+            </sphere>
+          </geometry>
+          <material>
+            <ambient>1 1 1 1</ambient>
+            <diffuse>1 1 1 1</diffuse>
+            <specular>1 1 1 1</specular>
+            <emissive>0 0 0 1</emissive>
+          </material>
+        </visual>
+    </link>
+    <joint name="light_joint" type="fixed">
+      <axis xyz="0 0 1" />
+      <origin xyz="-0.1 0 0.3" rpy="0 0 0"/>
+      <parent link="base_footprint"/>
+      <child link="light_link"/>
+    </joint>
+    <gazebo>
+      <plugin name="attach_light" filename="libAttachLightPlugin.so">
+          <link>
+              <link_name>light_link</link_name>
+              <light>
+                  <pose>0 0 0 0 0.785 0</pose>
+                  <light_name>light_source</light_name>
+              </light>
+          </link>
+      </plugin>
+    </gazebo>
 </robot>

File: turtlebot_gazebo/urdf/turtlebot3_burger_camera.urdf.xacro (robot description, xacro)
@@ -141,10 +141,65 @@
   </link>
   <link name="camera_link">
+    <visual>
+      <geometry>
+        <mesh filename="package://turtlebot_gazebo/models/r200/meshes/r200.dae"/>
+      </geometry>
+    </visual>
+    <collision>
+      <geometry>
+        <mesh filename="package://turtlebot_gazebo/models/r200/meshes/r200.dae" />
+      </geometry>
+    </collision>
+    <inertial>
+      <mass value="0.001" />
+	<inertia ixx="1" ixy="0.0" ixz="0.0"
+		 iyy="1" iyz="0.0"
+		 izz="1" />
+    </inertial>
   </link>
   <joint name="camera_joint" type="fixed">
     <axis xyz="0 0 1" />
-    <origin xyz="0 0 0.5" rpy="0 0 -0.707"/>
+    <origin xyz="0.04 0 0.14" rpy="1.5708 3.14159 1.5708"/>
     <parent link="base_footprint"/>
     <child link="camera_link"/>
   </joint>
+  <!-- **********************************************************-->
+  <!-- GAZEBO DEFINITIONS ***************************************-->
+  <gazebo reference ="camera_link">
+    <sensor type="camera" name="camera">
+      <update_rate>30.0</update_rate>
+      <camera name="head">
+	<pose>0 0 0 0 -1.5708 1.5708</pose>
+        <!--<horizontal_fov>1.3962634</horizontal_fov>-->
+        <image>
+          <width>1920</width>
+          <height>1080</height>
+          <format>R8G8B8</format>
+        </image>
+        <clip>
+          <near>0.02</near>
+          <far>300</far>
+        </clip>
+        <noise>
+            <type>gaussian</type>
+            <mean>0.0</mean>
+            <stddev>0.007</stddev>
+        </noise>
+      </camera>
+      <plugin name="camera_controller" filename="libgazebo_ros_camera.so">
+        <alwaysOn>true</alwaysOn>
+        <updateRate>0.0</updateRate>
+        <cameraName>raspicam_node</cameraName>
+        <imageTopicName>image_raw</imageTopicName>
+        <cameraInfoTopicName>camera_info</cameraInfoTopicName>
+        <frameName>camera_link</frameName>
+        <hackBaseline>0.0</hackBaseline>
+        <distortionK1>0.0</distortionK1>
+        <distortionK2>0.0</distortionK2>
+        <distortionK3>0.0</distortionK3>
+        <distortionT1>0.0</distortionT1>
+        <distortionT2>0.0</distortionT2>
+      </plugin>
+    </sensor>
+  </gazebo>
 </robot>
